File: hardware/dumper/dumper.kicad_pcb (KiCad board)
At the start: 2 copper layers, 90.2 x 55.9 mm, 27 parts, among them J1 /Reset, J10 arduino 10, J11 ss, J2 Clock In, J3 data, J4 clock, J5 2816 /WR disconnect, J6 arduino 13, J7 arduino 11, J8 arduino 5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

Commit message: added non-parallel rev. A with built in cmos detection
Other:
- board text added: "Ver. A"
- board text removed: "Ver. B"
Changed lines of the file:
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@@
     (effects (font (size 1 1) (thickness 0.15)) (justify mirror))
   )
-  (gr_text "Ver. B" (at 126.238 96.52) (layer "F.SilkS")
+  (gr_text "Ver. A" (at 126.238 96.52) (layer "F.SilkS")
     (effects (font (size 1 1) (thickness 0.15)))
   )
